Commit message: update urdf relative transform and still waiting for confirming imu data

File: xbot_description/urdf/sick_tim.urdf.xacro (robot description, xacro)
@@ -6,6 +6,6 @@
   <xacro:macro name="rplidarA2" params="name ros_topic">
     <xacro:sick_tim name="${name}" ros_topic="${ros_topic}"
-      length="0.06" width="0.06" height="0.079" mass="0.150" z_offset="0.05595"
-      min_range="0.2" max_range="8.0"
+      length="0.06" width="0.06" height="0.079" mass="0.150" z_offset="0.0308"
+      min_range="0.2" max_range="12.0"
       mesh="package://xbot_description/models/meshes/rplidar.dae" />
   </xacro:macro>

File: xbot_description/urdf/xbot-u.urdf.xacro (robot description, xacro)
@@ -66,5 +66,5 @@
     <parent link="base_link"/>
     <child link="laser_mount_link"/>
-    <origin rpy="0 0 0" xyz=".114 0 .17"/>
+    <origin rpy="0 0 0" xyz=".120 0 .205"/>
   </joint>
   <link name="imu_link"/>
@@ -73,5 +73,5 @@
     <parent link="base_link"/>
     <child link="imu_link"/>
-    <origin rpy="0 0 0" xyz="0 0 .2"/>
+    <origin rpy="0 0 0" xyz="0.0454 -0.0157 1.1724"/>
   </joint>
   <link name="left_wheel">
@@ -152,5 +152,5 @@
     <parent link="base_link"/>
     <child link="yaw_platform"/>
-    <origin rpy="0 0 0" xyz="0 0 1.305"/>
+    <origin rpy="0 0 0" xyz="0 0 1.232"/>
     <limit effort="100" velocity="100" lower="-1.57" upper="1.57" />
     <dynamics damping="0.0" friction="10.0"/>
@@ -179,5 +179,5 @@
     <parent link="yaw_platform"/>
     <child link="pitch_platform"/>
-    <origin rpy="0 0 0" xyz="0 0 0"/>
+    <origin rpy="0 0 0" xyz="0.0208 0 0.01325"/>
     <limit effort="100" velocity="100" lower="-1.57" upper="1.57" />
     <dynamics damping="0.0" friction="10.0"/>
