Commit message: v52版本在master上首次发布，加入机器人启动后播报功能

File: xbot_description/urdf/robot.xacro (robot description, xacro)
@@ -12,4 +12,4 @@
   <xacro:include filename="$(find xbot_description)/urdf/xbot-u.urdf.xacro" />
   <xacro:include filename="$(find xbot_description)/urdf/xbot-u.gazebo" />
-  <xacro:xbot2_base/>
+  <xacro:xbot_base/>
 </robot>

File: xbot_description/urdf/xbot-u.urdf.xacro (robot description, xacro)
@@ -4,5 +4,5 @@
   xmlns:sensor="http://playerstage.sourceforge.net/gazebo/xmlschema/#sensor"
   xmlns:xacro="http://ros.org/wiki/xacro">
-  <xacro:macro name="xbot2_base">
+  <xacro:macro name="xbot_base">
   <link name="base_footprint"/>
   <joint name="base_footprint_to_base" type="fixed">
